File: Peavey_5150.sch (KiCad schematic (older format))
At the start: 195 parts, among them J10 INPUT, J165 SEND, J166 RETURN, K2 G5V-2, K3 G5V-2, K4 G5V-2

Commit message: Add tube heat
Parts:
- added JP? (x5): PLS-2, symbol Device:Jumper_NC_Small
- added unit 3 of V1
- added unit 3 of V2
- added unit 3 of V3
- added unit 3 of V5
- added unit 3 of V6
Connections:
- net Earth: now also JP?.1, JP?.1
- net Earth_Protective: now also JP?.1, JP?.1, JP?.1
- net GND: now also V1.5 (F1), V2.5 (F1), V3.5 (F1), V5.5 (F1), V6.5 (F1)
- net HEAT+: now also V1.4 (F1), V2.4 (F1), V3.4 (F1), V5.4 (F1), V6.4 (F1)
- new net: JP?.2, V1.9 (F2)
- new net: JP?.2, V2.9 (F2)
- new net: JP?.2, V3.9 (F2)
- new net: JP?.2, V5.9 (F2)
- new net: JP?.2, V6.9 (F2)
Other:
- note added: "12.6V (6.3 for 6N2P)"
- note added: "Tube heat (put jumper for 6N2P)"
- note removed: "12.6V"

Commit message: add footswitch
Parts:
- removed K2, K4: G5V-2, symbol Relays:G5V-2
- added J?: FOOTSWITCH, symbol simple:Jack_6.35
- added K1, K2, K4, K5: G5V1, symbol Relays:G5V1
- added Q?: BC847, Package_TO_SOT_SMD:SOT-23, symbol Transistor_BJT:BC847
- added R?: 1K, symbol Device:R_US
- added R?: 10K, symbol Device:R_US
- added R?: 10, symbol Device:R_US
- added R? (x2): 47K, symbol Device:R_US
Connections:
- net +3V3: now also R?.2, R?.2
- net Earth: now also K1.5, K1.6, K5.5, K5.6
- net GND: now also J?.5, J?.6, Q?.2 (E), R?.1
- net HEAT+: no longer R?.2, R?.2
- net HEAT_IN: now also R?.2, R?.2, R?.2
- net MUTE: now also K2.5, K2.6
- net NRST: now also C?.1, U?.4 (NRST)
- net SWIM: now also U?.18 (PD1)
- net at C17.1, C6.2, R176.2: now also K4.5, K4.6
- net at C19.2, R40.1, R82.2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: now also K1.1
- net at C13.1: now also K4.10
- net at C51.1, R175.2, R19.2: now also K4.1
- net at C167.2: now also K1.10
- net at VR10.3: now also K2.10
- net at R?.1: now also K1.2, K2.2
- net at Q?.3 (C): now also K1.9, K2.9
- net at VR5.3: now also K2.1
- net at C63.2, R174.2: now also K5.1
- net at R?.1: now also K4.2, K5.2
- net at Q?.3 (C): now also K4.9, K5.9
- net at C155.1, R163.2: now also K5.10
- net SEND_RETURN: now reaches U?.1 (PD4)
- net SEND_RETURN: now also R?.2
- net FS2: now reaches U?.11 (PB5)
- net FS2: now also J?.1, J?.2, R?.1
- net FS1: now reaches U?.12 (PB4)
- net FS1: now also J?.3, J?.4, R?.1
- net at K3.1: now also R?.1
- net at K3.16: now also Q?.3 (C)
- new net: Q?.1 (B), R?.1, R?.2
- no-connect marks 16 -> 12
Other:
- moved on the sheet: C?, K3A, R?

Commit message: Split schematic
Parts:
- added K?: G5V1, symbol Relays:G5V1
- added R? (x2): 47R1W, symbol Device:R_US
- added SW?: Ultra, symbol Switch:SW_Push
- added SW?: Clean, symbol Switch:SW_Push
- added SW?: Crunch, symbol Switch:SW_Push
- added SW?: FX_loop, symbol Switch:SW_Push
Connections:
- net Earth: now also K?.5, K?.6, R?.2
- net Earth_Protective: now also R?.1, R?.2
- net GNDPWR: now also R?.1
- net at C19.2, R40.1, R82.2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: now also K?.1; no longer K1.1
Changed lines of the file:
@@
 Connection ~ 5800 5800
 Wire Wire Line
-	6400 3900 6500 3900
-Wire Wire Line
-	6500 3900 6500 5800
+	6500 4500 6500 5800
 Wire Wire Line
 	6500 5800 6050 5800
@@
 Text Label 23150 13600 0    50   ~ 0
 FS2
+$Comp
+L power:Earth_Protective #PWR?
+U 1 1 5E166149
+P 15650 1950
+F 0 "#PWR?" H 15900 1700 50  0001 C CNN
+F 1 "Earth_Protective" H 16100 1800 50  0001 C CNN
+F 2 "" H 15650 1850 50  0001 C CNN
+F 3 "~" H 15650 1850 50  0001 C CNN
+	1    15650 1950
+	1    0    0    -1
+$EndComp
+$Comp
+L power:Earth #PWR?
+U 1 1 5E166622
+P 15150 1950
+F 0 "#PWR?" H 15150 1700 50  0001 C CNN
+F 1 "Earth" H 15150 1800 50  0001 C CNN
+F 2 "" H 15150 1950 50  0001 C CNN
+F 3 "~" H 15150 1950 50  0001 C CNN
+	1    15150 1950
+	1    0    0    -1
+$EndComp
+Text Label 16150 1850 0    50   ~ 0
+GNDPWR
+$Comp
+L Device:R_US R?
+U 1 1 5E167781
+P 15900 1850
+F 0 "R?" V 15800 1850 50  0000 C CNN
+F 1 "47R1W" V 16000 1850 50  0000 C CNN
+F 2 "" V 15940 1840 50  0001 C CNN
+F 3 "~" H 15900 1850 50  0001 C CNN
+	1    15900 1850
+	0    1    1    0
+$EndComp
+Wire Wire Line
+	16050 1850 16150 1850
+Wire Wire Line
+	15750 1850 15650 1850
+Wire Wire Line
+	15650 1850 15650 1950
+$Comp
+L Device:R_US R?
+U 1 1 5E22F05E
+P 15400 1850
+F 0 "R?" V 15300 1850 50  0000 C CNN
+F 1 "47R1W" V 15500 1850 50  0000 C CNN
+F 2 "" V 15440 1840 50  0001 C CNN
+F 3 "~" H 15400 1850 50  0001 C CNN
+	1    15400 1850
+	0    1    1    0
+$EndComp
+Wire Wire Line
+	15650 1850 15550 1850
+Connection ~ 15650 1850
+Wire Wire Line
+	15250 1850 15150 1850
+Wire Wire Line
+	15150 1850 15150 1950
+$Comp
+L Switch:SW_Push SW?
+U 1 1 5E2FB160
+P 24250 13700
+F 0 "SW?" V 24204 13848 50  0000 L CNN
+F 1 "Ultra" V 24295 13848 50  0000 L CNN
+F 2 "" H 24250 13900 50  0001 C CNN
+F 3 "~" H 24250 13900 50  0001 C CNN
+	1    24250 13700
+	0    1    1    0
+$EndComp
+$Comp
+L Switch:SW_Push SW?
+U 1 1 5E2FC3AC
+P 24900 13700
+F 0 "SW?" V 24854 13848 50  0000 L CNN
+F 1 "Clean" V 24945 13848 50  0000 L CNN
+F 2 "" H 24900 13900 50  0001 C CNN
+F 3 "~" H 24900 13900 50  0001 C CNN
+	1    24900 13700
+	0    1    1    0
+$EndComp
+$Comp
+L Switch:SW_Push SW?
+U 1 1 5E2FC968
+P 25550 13700
+F 0 "SW?" V 25504 13848 50  0000 L CNN
+F 1 "Crunch" V 25595 13848 50  0000 L CNN
+F 2 "" H 25550 13900 50  0001 C CNN
+F 3 "~" H 25550 13900 50  0001 C CNN
+	1    25550 13700
+	0    1    1    0
+$EndComp
+$Comp
+L Switch:SW_Push SW?
+U 1 1 5E2FCF10
+P 26200 13700
+F 0 "SW?" V 26154 13848 50  0000 L CNN
+F 1 "FX_loop" V 26245 13848 50  0000 L CNN
+F 2 "" H 26200 13900 50  0001 C CNN
+F 3 "~" H 26200 13900 50  0001 C CNN
+	1    26200 13700
+	0    1    1    0
+$EndComp
+Wire Notes Line
+	8050 1050 5100 1050
+Wire Notes Line
+	5100 1050 5100 2100
+Wire Notes Line
+	5100 2100 5650 2100
+Wire Notes Line
+	5650 2100 5650 3100
+$Comp
+L Relays:G5V1 K?
+U 2 1 5E362714
+P 6150 4400
+F 0 "K?" H 6100 4119 50  0000 C CNN
+F 1 "G5V1" H 6100 4210 50  0000 C CNN
+F 2 "" H 6150 4400 50  0001 C CNN
+F 3 "" H 6150 4400 50  0001 C CNN
+	2    6150 4400
+	1    0    0    1
+$EndComp
+$Comp
+L power:Earth #PWR?
+U 1 1 5E3645A3
+P 5700 4500
+F 0 "#PWR?" H 5700 4250 50  0001 C CNN
+F 1 "Earth" H 5700 4350 50  0001 C CNN
+F 2 "" H 5700 4500 50  0001 C CNN
+F 3 "~" H 5700 4500 50  0001 C CNN
+	1    5700 4500
+	1    0    0    -1
+$EndComp
+Wire Wire Line
+	5800 4400 5700 4400
+Wire Wire Line
+	5700 4400 5700 4500
+Wire Wire Line
+	5800 4300 5700 4300
+Wire Wire Line
+	5700 4300 5700 4400
+Connection ~ 5700 4400
+Wire Wire Line
+	6500 4500 6400 4500
+Wire Notes Line
+	5500 3100 5500 4050
+Wire Notes Line
+	5500 4050 8050 4050
+Wire Notes Line
+	8050 1050 8050 4050
+Wire Notes Line
+	5500 3100 5650 3100
+Wire Notes Line
+	10500 2550 11150 2550
+Wire Notes Line
+	11150 2550 11150 700
+Wire Notes Line
+	11150 700  14150 700
+Wire Notes Line
+	14150 700  14150 4400
+Wire Notes Line
+	14150 4400 10100 4400
+Wire Notes Line
+	10100 4400 10100 2950
+Wire Notes Line
+	10100 2950 10500 2950
+Wire Notes Line
+	10500 2950 10500 2550
 $EndSCHEMATC

Commit message: Separate
Parts:
- added C?: 22uF, symbol Device:CP1
Connections:
- net GND: now also C?.1
- net K4B_56: now reaches C17.1, C6.2, K4.5, K4.6, R176.2
- net V6A_7: now reaches C151.2, R152.1, R154.2, V6.7 (G)
- net at C38.2, C?.1, C?.2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: now also C?.2
- net C153_2: now reaches C153.2, R153.2, R75.2
- net K2B_1: now reaches K2.1, VR5.3
Other:
- moved on the sheet: C1, C10, C11, C13, C14, C15, C150, C151, C152, C153, C154, C155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

Commit message: add V3
Parts:
- removed V? (x2): V1+, symbol simple:V1+
- added C? (x3): 22uF, symbol Device:CP1
- added R? (x2): 10K 1W, symbol Device:R_US
- added R?: 5K1 1W, symbol Device:R_US
- added U?: LT1129-3.3_SOT223, Package_TO_SOT_SMD:SOT-223-3_TabPin2, symbol Regulator_Linear:LT1129-3.3_SOT223
- added V3? (x2), V?: V3+, symbol simple:V3+
- added V?: V1+, symbol simple:V1+
- added V?: V2+, symbol simple:V2+
Connections:
- net Earth: now also C?.2, C?.2
- net Earth_Protective: now also C?.2
- net V1+: now also C?.1, C?.1, C?.1, R?.1, R?.1, R?.1, R?.2, R?.2, V3?.1 (V1+), V3?.1 (V1+), V?.1 (V1+), V?.1 (V1+), V?.1 (V1+)
- net at C?.1, Q?.3 (S), R?.2: now also R?.2
Changed lines of the file:
@@
 	-1   0    0    1
 $EndComp
-$Comp
-L simple:V1+ V?
-U 1 1 5DE60FCC
-P 8500 5800
-F 0 "V?" H 8600 5850 50  0001 C CNN
-F 1 "V1+" H 8450 5950 50  0000 L CNN
-F 2 "" H 8500 5800 50  0001 C CNN
-F 3 "" H 8500 5800 50  0001 C CNN
-	1    8500 5800
-	1    0    0    -1
-$EndComp
 Wire Wire Line
 	8500 6500 8500 6200
@@
 $EndComp
 $Comp
-L simple:V1+ V?
-U 1 1 5DF899F2
-P 9750 5800
-F 0 "V?" H 9850 5850 50  0001 C CNN
-F 1 "V1+" H 9700 5950 50  0000 L CNN
-F 2 "" H 9750 5800 50  0001 C CNN
-F 3 "" H 9750 5800 50  0001 C CNN
-	1    9750 5800
-	1    0    0    -1
-$EndComp
-$Comp
 L Device:R_US R171
 U 1 1 5DF89FD7
@@
 Wire Notes Line
 	4600 4850 14150 4850
+$Comp
+L Regulator_Linear:LT1129-3.3_SOT223 U?
+U 1 1 5E37AA6F
+P 15850 14250
+F 0 "U?" H 15850 14492 50  0000 C CNN
+F 1 "LT1129-3.3_SOT223" H 15850 14401 50  0000 C CNN
+F 2 "Package_TO_SOT_SMD:SOT-223-3_TabPin2" H 15850 14475 50  0001 C CIN
+F 3 "https://www.analog.com/media/en/technical-documentation/data-sheets/112935ff.pdf" H 15850 14200 50  0001 C CNN
+	1    15850 14250
+	1    0    0    -1
+$EndComp
+$Comp
+L Device:CP1 C?
+U 1 1 5E607A3D
+P 13400 14550
+F 0 "C?" H 13500 14600 50  0000 L CNN
+F 1 "22uF" H 13500 14500 50  0000 L CNN
+F 2 "" H 13400 14550 50  0001 C CNN
+F 3 "~" H 13400 14550 50  0001 C CNN
+	1    13400 14550
+	1    0    0    -1
+$EndComp
+$Comp
+L Device:R_US R?
+U 1 1 5E60CBF9
+P 13850 14300
+F 0 "R?" V 13750 14300 50  0000 C CNN
+F 1 "10K 1W" V 13950 14300 50  0000 C CNN
+F 2 "" V 13890 14290 50  0001 C CNN
+F 3 "~" H 13850 14300 50  0001 C CNN
+	1    13850 14300
+	0    1    1    0
+$EndComp
+Wire Wire Line
+	13700 14300 13400 14300
+Wire Wire Line
+	13400 14400 13400 14300
+$Comp
+L Device:CP1 C?
+U 1 1 5E75E672
+P 14250 14550
+F 0 "C?" H 14350 14600 50  0000 L CNN
+F 1 "22uF" H 14350 14500 50  0000 L CNN
+F 2 "" H 14250 14550 50  0001 C CNN
+F 3 "~" H 14250 14550 50  0001 C CNN
+	1    14250 14550
+	1    0    0    -1
+$EndComp
+$Comp
+L Device:R_US R?
+U 1 1 5E75F963
+P 13050 14300
+F 0 "R?" V 12950 14300 50  0000 C CNN
+F 1 "5K1 1W" V 13150 14300 50  0000 C CNN
+F 2 "" V 13090 14290 50  0001 C CNN
+F 3 "~" H 13050 14300 50  0001 C CNN
+	1    13050 14300
+	0    1    1    0
+$EndComp
+Wire Wire Line
+	12900 14300 11950 14300
+Connection ~ 11950 14300
+Wire Wire Line
+	13400 14300 13200 14300
+Connection ~ 13400 14300
+Wire Wire Line
+	14250 14400 14250 14300
+Wire Wire Line
+	14250 14300 14000 14300
+$Comp
+L simple:V1+ V?
+U 1 1 5E8B2C7F
+P 14250 14200
+F 0 "V?" H 14350 14250 50  0001 C CNN
+F 1 "V1+" H 14200 14350 50  0000 L CNN
+F 2 "" H 14250 14200 50  0001 C CNN
+F 3 "" H 14250 14200 50  0001 C CNN
+	1    14250 14200
+	1    0    0    -1
+$EndComp
+Wire Wire Line
+	14250 14200 14250 14300
+Connection ~ 14250 14300
+$Comp
+L power:Earth_Protective #PWR?
+U 1 1 5E924C43
+P 13400 14800
+F 0 "#PWR?" H 13650 14550 50  0001 C CNN
+F 1 "Earth_Protective" H 13850 14650 50  0001 C CNN
+F 2 "" H 13400 14700 50  0001 C CNN
+F 3 "~" H 13400 14700 50  0001 C CNN
+	1    13400 14800
+	1    0    0    -1
+$EndComp
+Wire Wire Line
+	13400 14800 13400 14700
+$Comp
+L power:Earth #PWR?
+U 1 1 5E997673
+P 14250 14800
+F 0 "#PWR?" H 14250 14550 50  0001 C CNN
+F 1 "Earth" H 14250 14650 50  0001 C CNN
+F 2 "" H 14250 14800 50  0001 C CNN
+F 3 "~" H 14250 14800 50  0001 C CNN
+	1    14250 14800
+	1    0    0    -1
+$EndComp
+Wire Wire Line
+	14250 14800 14250 14700
+$Comp
+L simple:V2+ V?
+U 1 1 5EA0A2A4
+P 13400 13150
+F 0 "V?" H 13500 13200 50  0001 C CNN
+F 1 "V2+" H 13350 13300 50  0000 L CNN
+F 2 "" H 13400 13150 50  0001 C CNN
+F 3 "" H 13400 13150 50  0001 C CNN
+	1    13400 13150
+	1    0    0    -1
+$EndComp
+Wire Wire Line
+	13400 13150 13400 13250
+$Comp
+L simple:V3+ V3?
+U 1 1 5EA8D447
+P 9750 5700
+F 0 "V3?" H 9850 5750 50  0001 C CNN
+F 1 "V3+" H 9700 5850 50  0000 L CNN
+F 2 "" H 9750 5700 50  0001 C CNN
+F 3 "" H 9750 5700 50  0001 C CNN
+	1    9750 5700
+	1    0    0    -1
+$EndComp
+$Comp
+L simple:V3+ V?
+U 1 1 5EA8FC50
+P 8500 5700
+F 0 "V?" H 8600 5750 50  0001 C CNN
+F 1 "V3+" H 8450 5850 50  0000 L CNN
+F 2 "" H 8500 5700 50  0001 C CNN
+F 3 "" H 8500 5700 50  0001 C CNN
+	1    8500 5700
+	1    0    0    -1
+$EndComp
+Wire Wire Line
+	9750 5700 9750 5800
+Wire Wire Line
+	8500 5700 8500 5800
+$Comp
+L simple:V3+ V3?
+U 1 1 5EB761EE
+P 14250 13150
+F 0 "V3?" H 14350 13200 50  0001 C CNN
+F 1 "V3+" H 14200 13300 50  0000 L CNN
+F 2 "" H 14250 13150 50  0001 C CNN
+F 3 "" H 14250 13150 50  0001 C CNN
+	1    14250 13150
+	1    0    0    -1
+$EndComp
+$Comp
+L Device:R_US R?
+U 1 1 5EB789BC
+P 13850 13250
+F 0 "R?" V 13750 13250 50  0000 C CNN
+F 1 "10K 1W" V 13950 13250 50  0000 C CNN
+F 2 "" V 13890 13240 50  0001 C CNN
+F 3 "~" H 13850 13250 50  0001 C CNN
+	1    13850 13250
+	0    1    1    0
+$EndComp
+Wire Wire Line
+	13700 13250 13400 13250
+Connection ~ 13400 13250
+Wire Wire Line
+	13400 13250 13400 14300
+$Comp
+L Device:CP1 C?
+U 1 1 5ECD1800
+P 14250 13500
+F 0 "C?" H 14350 13550 50  0000 L CNN
+F 1 "22uF" H 14350 13450 50  0000 L CNN
+F 2 "" H 14250 13500 50  0001 C CNN
+F 3 "~" H 14250 13500 50  0001 C CNN
+	1    14250 13500
+	1    0    0    -1
+$EndComp
+Wire Wire Line
+	14000 13250 14250 13250
+Wire Wire Line
+	14250 13250 14250 13350
+Wire Wire Line
+	14250 13250 14250 13150
+Connection ~ 14250 13250
+$Comp
+L power:Earth #PWR?
+U 1 1 5EDBC158
+P 14250 13750
+F 0 "#PWR?" H 14250 13500 50  0001 C CNN
+F 1 "Earth" H 14250 13600 50  0001 C CNN
+F 2 "" H 14250 13750 50  0001 C CNN
+F 3 "~" H 14250 13750 50  0001 C CNN
+	1    14250 13750
+	1    0    0    -1
+$EndComp
+Wire Wire Line
+	14250 13750 14250 13650
 $EndSCHEMATC

Commit message: AMS1117-3.3
Parts:
- added C? (x2): 1uF, symbol simple:C_US
- added unit 1 of K6
- U?: value LT1129-3.3_SOT223 -> AMS1117-3.3
- gave numbers to parts that had none: 1
Connections:
- net +3V3: now also U?.3 (VO), C?.1
- net GND: now also U?.2 (GND), C?.2, C?.2
- net HEAT+: now also U?.1 (VI), C?.1
- net at K1.2, K2.2, R?.1: now also K6.2
- net at K1.9, K2.9, Q?.3 (C): now also K6.9
- no-connect marks 12 -> 14
Other:
- moved on the sheet: U?
Changed lines of the file:
@@
 $EndComp
 $Comp
-L Relays:G5V1 K?
+L Relays:G5V1 K6
 U 2 1 5E362714
 P 6000 8600
-F 0 "K?" H 5950 8319 50  0000 C CNN
+F 0 "K6" H 5950 8319 50  0000 C CNN
 F 1 "G5V1" H 5950 8410 50  0000 C CNN
 F 2 "" H 6000 8600 50  0001 C CNN
@@
 L Regulator_Linear:LT1129-3.3_SOT223 U?
 U 1 1 5E37AA6F
-P 15850 14250
-F 0 "U?" H 15850 14492 50  0000 C CNN
-F 1 "LT1129-3.3_SOT223" H 15850 14401 50  0000 C CNN
-F 2 "Package_TO_SOT_SMD:SOT-223-3_TabPin2" H 15850 14475 50  0001 C CIN
-F 3 "https://www.analog.com/media/en/technical-documentation/data-sheets/112935ff.pdf" H 15850 14200 50  0001 C CNN
-	1    15850 14250
+P 15050 17550
+F 0 "U?" H 15050 17792 50  0000 C CNN
+F 1 "AMS1117-3.3" H 15050 17701 50  0000 C CNN
+F 2 "Package_TO_SOT_SMD:SOT-223-3_TabPin2" H 15050 17775 50  0001 C CIN
+F 3 "https://www.analog.com/media/en/technical-documentation/data-sheets/112935ff.pdf" H 15050 17500 50  0001 C CNN
+	1    15050 17550
 	1    0    0    -1
 $EndComp
@@
 Wire Wire Line
 	14250 13750 14250 13650
+$Comp
+L power:GND #PWR?
+U 1 1 5EBFDBD4
+P 15050 18050
+F 0 "#PWR?" H 15050 17800 50  0001 C CNN
+F 1 "GND" H 15055 17877 50  0000 C CNN
+F 2 "" H 15050 18050 50  0001 C CNN
+F 3 "" H 15050 18050 50  0001 C CNN
+	1    15050 18050
+	1    0    0    -1
+$EndComp
+$Comp
+L power:+3V3 #PWR?
+U 1 1 5EC01E4E
+P 15450 17450
+F 0 "#PWR?" H 15450 17300 50  0001 C CNN
+F 1 "+3V3" H 15465 17623 50  0000 C CNN
+F 2 "" H 15450 17450 50  0001 C CNN
+F 3 "" H 15450 17450 50  0001 C CNN
+	1    15450 17450
+	1    0    0    -1
+$EndComp
+Wire Wire Line
+	14750 17550 14650 17550
+Text Label 14550 17550 2    50   ~ 0
+HEAT+
+$Comp
+L Relays:G5V1 K6
+U 1 1 5EC89CFC
+P 23700 15100
+F 0 "K6" H 23855 15146 50  0000 L CNN
+F 1 "G5V1" H 23855 15055 50  0000 L CNN
+F 2 "" H 23700 15100 50  0001 C CNN
+F 3 "" H 23700 15100 50  0001 C CNN
+	1    23700 15100
+	1    0    0    -1
+$EndComp
+Wire Wire Line
+	23700 15400 23700 15500
+Wire Wire Line
+	23700 15500 23150 15500
+Wire Wire Line
+	23700 14800 23700 14700
+Wire Wire Line
+	23700 14700 23150 14700
+NoConn ~ 6300 4350
+NoConn ~ 6250 8500
+Wire Wire Line
+	15050 18050 15050 17850
+Wire Wire Line
+	15350 17550 15450 17550
+Wire Wire Line
+	15450 17550 15450 17450
+$Comp
+L simple:C_US C?
+U 1 1 5EF50F2E
+P 15450 17800
+F 0 "C?" H 15350 17850 50  0000 R CNN
+F 1 "1uF" H 15350 17750 50  0000 R CNN
+F 2 "" H 15450 17800 50  0001 C CNN
+F 3 "" H 15450 17800 50  0001 C CNN
+	1    15450 17800
+	-1   0    0    -1
+$EndComp
+Connection ~ 15450 17550
+Wire Wire Line
+	15450 17650 15450 17550
+$Comp
+L power:GND #PWR?
+U 1 1 5EFCA80A
+P 15450 18050
+F 0 "#PWR?" H 15450 17800 50  0001 C CNN
+F 1 "GND" H 15455 17877 50  0000 C CNN
+F 2 "" H 15450 18050 50  0001 C CNN
+F 3 "" H 15450 18050 50  0001 C CNN
+	1    15450 18050
+	1    0    0    -1
+$EndComp
+Wire Wire Line
+	15450 18050 15450 17950
+$Comp
+L simple:C_US C?
+U 1 1 5F0B9F5F
+P 14650 17800
+F 0 "C?" H 14550 17850 50  0000 R CNN
+F 1 "1uF" H 14550 17750 50  0000 R CNN
+F 2 "" H 14650 17800 50  0001 C CNN
+F 3 "" H 14650 17800 50  0001 C CNN
+	1    14650 17800
+	1    0    0    -1
+$EndComp
+Wire Wire Line
+	14650 17650 14650 17550
+Connection ~ 14650 17550
+Wire Wire Line
+	14650 17550 14550 17550
+$Comp
+L power:GND #PWR?
+U 1 1 5F1AAF4D
+P 14650 18050
+F 0 "#PWR?" H 14650 17800 50  0001 C CNN
+F 1 "GND" H 14655 17877 50  0000 C CNN
+F 2 "" H 14650 18050 50  0001 C CNN
+F 3 "" H 14650 18050 50  0001 C CNN
+	1    14650 18050
+	1    0    0    -1
+$EndComp
+Wire Wire Line
+	14650 18050 14650 17950
 $EndSCHEMATC

Commit message: Add protection diodes to relay
Parts:
- removed unit 2 of K1
- removed unit 1 of K6
- removed V2?, V? (x5): V2+, symbol simple:V2+
- removed V3? (x2), V?: V3+, symbol simple:V3+
- removed V? (x4): V1+, symbol simple:V1+
- added C42, C43, C44, C45: 0.1uF, symbol simple:C_US
- added D3, D4, D6: WHITE, symbol Device:LED
- added D5: RED, symbol Device:LED
- added D7, D8, D9: D, symbol Device:D
- added J6, J7: IDC-10, symbol Connector_Generic:Conn_02x05_Odd_Even
- added R53: 200, symbol Device:R_US
- added R54, R55, R56, R57: 47K, symbol Device:R_US
- added R58, R59, R60, R61: 1K, symbol Device:R_US
- added R63: 47R1W, symbol Device:R_US
- added U4: TLP222A, Package_DIP:DIP-4_W7.62mm, symbol Relay_SolidState:TLP222A
- gave numbers to parts that had none: 80
- renumbered C4 to C48, K6 to K1
Connections:
- net PE is gone; now on net GNDPWR: J2.2 (Pin_2)
- net +3V3: now also R54.2, R55.2, R56.2, R57.2
- net ASWA: now also R35.1
- net ASWB: now also C30.1, R37.2, R38.2, R4.2, R5.2, R86.2, R96.2, V3.6 (A)
- net C153_2: now also J7.5 (Pin_5); no longer R153.2, R75.2
- net DIST_CLEAN: now also R60.2
- net Earth: now also J7.7 (Pin_7), J7.8 (Pin_8); no longer C157.2, C31.2, K5.5, K5.6, R154.1, R158.1, VR1.1
- net Earth_Protective: now also R63.1, U4.4; no longer C166.2, R155.1, R156.1, R159.1, R172.1, VR3.1, VR5.1
- net GND: now also SW1.2, SW2.2, SW3.2, SW4.2, C42.2, C43.2, C44.2, C45.2, D3.1 (K), D4.1 (K), D5.1 (K), D6.1 (K), U4.2
- net K2B_1: now also J7.6 (Pin_6); no longer VR5.3
- net MUTE: now also U3.20 (PD3), R53.2; no longer C52.1, K2.5, K2.6, R81.2
- net SEND_RETURN: now also R61.2
- net V1+: no longer C30.1, C31.1, R150.2, R170.2, R35.1, R37.1, R37.2, R38.2, R4.2, R5.2, R86.2, R96.2, V3.6 (A)
- net V6A_7: now also J7.4 (Pin_4); no longer C151.2, R152.1
- net С27_TOP: now reaches C27.1, R174.1, R23.1, VR1.2
- net С27_TOP: now also J6.3 (Pin_3); no longer C13.2, C51.2, R19.1
- net at C167.2: now also K1.10
- net ULTRA_B: now reaches SW1.1
- net ULTRA_B: now also U3.15 (PC5), C44.1, R56.1
- net CLEAN_B: now reaches SW2.1
- net CLEAN_B: now also U3.13 (PC3), C42.1, R54.1
- net CRUNCH_B: now reaches SW3.1
- net CRUNCH_B: now also U3.14 (PC4), C43.1, R55.1
- net FX_LOOP_B: now reaches SW4.1
- net FX_LOOP_B: now also U3.16 (PC6), C45.1, R57.1
- net at K1.2, K2.2, R46.1: now also D7.1 (K)
- net at K1.9, K2.9, Q2.3 (C): now also D7.2 (A)
- net K5A_2: now reaches K4.2, R49.1
- net K5A_2: now also D8.1 (K), J7.10 (Pin_10); no longer K5.2
- net K5A_9: now reaches K4.9, Q3.3 (C)
- net K5A_9: now also D8.2 (A), J7.9 (Pin_9); no longer K5.9
- net CRUNCH_LED: now reaches U3.17 (PC7)
- net CRUNCH_LED: now also R59.2
- net CLEAN_LED: now reaches U3.19 (PD2)
- net CLEAN_LED: now also R58.2
- net at K3.1, R52.1: now also D9.1 (K)
- net at K3.16, Q4.3 (C): now also D9.2 (A)
- net K4B_56: no longer names the net of C17.1, C6.2, K4.5, K4.6, R176.2
- new net: C52.1, K2.5, K2.6, R81.2, U4.3
- new net: R53.1, U4.1
- new net: D6.2 (A), R61.1
- new net: D5.2 (A), R60.1
- new net: D4.2 (A), R59.1
- new net: D3.2 (A), R58.1
- new net C153_2_TOP: J6.5 (Pin_5), R153.2, R75.2
- new net GND_V1_TOP: J6.7 (Pin_7), J6.8 (Pin_8), K5.5, K5.6
- new net GND_V3: C157.2, C166.2, C31.2, J7.1 (Pin_1), J7.2 (Pin_2), R154.1, R155.1, R158.1, R172.1, R63.2
- new net GND_V3_TOP: J6.1 (Pin_1), J6.2 (Pin_2), R156.1, R159.1, VR1.1, VR3.1, VR5.1
- new net K2B_1_TOP: J6.6 (Pin_6), VR5.3
- new net K5A_2_TOP: J6.10 (Pin_10), K5.2
- new net K5A_9_TOP: J6.9 (Pin_9), K5.9
- new net V3+: C31.1, R150.2, R170.2, R37.1
- new net V6A_7_TOP: C151.2, J6.4 (Pin_4), R152.1
- new net С27: C13.2, C51.2, J7.3 (Pin_3), R19.1
- no-connect marks 14 -> 5
Other:
- note added: "10..15mA"
- moved on the sheet: C10, C13, C150, C151, C152, C154, C155, C156, C157, C167, C27, C51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

Commit message: Fix ground on clean part Change board connector to KF2510
Parts:
- removed J6, J7: IDC-10, symbol Connector_Generic:Conn_02x05_Odd_Even
- added J6, J7, J8, J9: KF2510, symbol Connector_Generic:Conn_01x04
Connections:
- net GND_V1_TOP is gone; now on net GND_V3_TOP: K5.5, K5.6
- net C153_2: now also J9.1 (Pin_1)
- net C153_2_TOP: now also J7.1 (Pin_1)
- net Earth: no longer C48.2, C5.2, R101.1, R102.1, R11.1, R13.1, R91.1
- net Earth_Protective: now also C48.2, C5.2, R101.1, R102.1, R11.1, R13.1, R91.1
- net GND_V3: now also J8.1 (Pin_1), J8.2 (Pin_2)
- net GND_V3_TOP: now also J6.1 (Pin_1), J6.2 (Pin_2)
- net K2B_1: now also J9.2 (Pin_2)
- net K2B_1_TOP: now also J7.2 (Pin_2)
- net K5A_2: now also J9.3 (Pin_3)
- net K5A_2_TOP: now also J7.3 (Pin_3)
- net K5A_9: now also J9.4 (Pin_4)
- net K5A_9_TOP: now also J7.4 (Pin_4)
- net V6A_7: now also J8.4 (Pin_4)
- net V6A_7_TOP: now also J6.4 (Pin_4)
- net С27: now also J8.3 (Pin_3)
- net С27_TOP: now also J6.3 (Pin_3)
Other:
- moved on the sheet: K3C, R176
